Commit message: feat: gz sim  roma import

File: roma_description/urdf/roma.urdf (robot description, URDF)
Before this commit: robot roma, 13 links, 12 joints
Joints:
- joint wheel_left_front_link_joint: limit effort=0.0000 velocity=0.0000 -> effort=10.0000 velocity=20.0000
- joint wheel_left_rear_link_joint: limit effort=0.0000 velocity=0.0000 -> effort=10.0000 velocity=20.0000
- joint wheel_right_front_link_joint: limit effort=0.0000 velocity=0.0000 -> effort=10.0000 velocity=20.0000
- joint wheel_right_rear_link_joint: limit effort=0.0000 velocity=0.0000 -> effort=10.0000 velocity=20.0000

File: roma_description/urdf/roma.urdf.xacro (robot description, xacro)
@@ -1,23 +1,25 @@
 <?xml version="1.0"?>
 <robot name="roma" xmlns:xacro="http://www.ros.org/wiki/xacro">
-<!-- Properties -->
-  <xacro:property name="visual_mesh_dir" value="package://roma_description/meshes/visual"/>
-  <xacro:property name="collision_mesh_dir" value="package://roma_description/meshes/collision"/>
-  <xacro:property name="mesh_scale" value="1 1 1"/>
-<!-- Reusable macros -->
+  <!-- Properties -->
+  <!-- Mesh path configuration -->
+  <xacro:arg name="mesh_uri_prefix" default="package://roma_description" />
+  <xacro:property name="visual_mesh_dir" value="$(arg mesh_uri_prefix)/meshes/visual" />
+  <xacro:property name="collision_mesh_dir" value="$(arg mesh_uri_prefix)/meshes/collision" />
+  <xacro:property name="mesh_scale" value="1 1 1" />
+  <!-- Reusable macros -->
   <xacro:macro name="mesh_visual" params="name mesh material xyz rpy">
     <visual name="${name}">
-      <origin xyz="${xyz}" rpy="${rpy}"/>
+      <origin xyz="${xyz}" rpy="${rpy}" />
       <geometry>
-        <mesh filename="${mesh}" scale="${mesh_scale}"/>
+        <mesh filename="${mesh}" scale="${mesh_scale}" />
       </geometry>
-      <material name="${material}"/>
+      <material name="${material}" />
     </visual>
   </xacro:macro>
   <xacro:macro name="mesh_collision" params="name mesh xyz rpy">
     <collision name="${name}">
-      <origin xyz="${xyz}" rpy="${rpy}"/>
+      <origin xyz="${xyz}" rpy="${rpy}" />
       <geometry>
-        <mesh filename="${mesh}" scale="${mesh_scale}"/>
+        <mesh filename="${mesh}" scale="${mesh_scale}" />
       </geometry>
     </collision>
@@ -25,42 +27,43 @@
   <xacro:macro name="link_inertial" params="mass xyz rpy ixx ixy ixz iyy iyz izz">
     <inertial>
-      <origin xyz="${xyz}" rpy="${rpy}"/>
-      <mass value="${mass}"/>
-      <inertia ixx="${ixx}" ixy="${ixy}" ixz="${ixz}" iyy="${iyy}" iyz="${iyz}" izz="${izz}"/>
+      <origin xyz="${xyz}" rpy="${rpy}" />
+      <mass value="${mass}" />
+      <inertia ixx="${ixx}" ixy="${ixy}" ixz="${ixz}" iyy="${iyy}" iyz="${iyz}" izz="${izz}" />
     </inertial>
   </xacro:macro>
   <xacro:macro name="fixed_joint" params="name parent child xyz rpy">
     <joint name="${name}" type="fixed">
-      <origin xyz="${xyz}" rpy="${rpy}"/>
-      <parent link="${parent}"/>
-      <child link="${child}"/>
+      <origin xyz="${xyz}" rpy="${rpy}" />
+      <parent link="${parent}" />
+      <child link="${child}" />
     </joint>
   </xacro:macro>
-  <xacro:macro name="revolute_joint" params="name parent child xyz rpy axis lower upper effort velocity">
+  <xacro:macro name="revolute_joint"
+    params="name parent child xyz rpy axis lower upper effort velocity">
     <joint name="${name}" type="revolute">
-      <origin xyz="${xyz}" rpy="${rpy}"/>
-      <parent link="${parent}"/>
-      <child link="${child}"/>
-      <axis xyz="${axis}"/>
-      <limit lower="${lower}" upper="${upper}" effort="${effort}" velocity="${velocity}"/>
+      <origin xyz="${xyz}" rpy="${rpy}" />
+      <parent link="${parent}" />
+      <child link="${child}" />
+      <axis xyz="${axis}" />
+      <limit lower="${lower}" upper="${upper}" effort="${effort}" velocity="${velocity}" />
     </joint>
   </xacro:macro>
   <xacro:macro name="continuous_joint" params="name parent child xyz rpy axis effort velocity">
     <joint name="${name}" type="continuous">
-      <origin xyz="${xyz}" rpy="${rpy}"/>
-      <parent link="${parent}"/>
-      <child link="${child}"/>
-      <axis xyz="${axis}"/>
-      <limit effort="${effort}" velocity="${velocity}"/>
+      <origin xyz="${xyz}" rpy="${rpy}" />
+      <parent link="${parent}" />
+      <child link="${child}" />
+      <axis xyz="${axis}" />
+      <limit effort="${effort}" velocity="${velocity}" />
     </joint>
   </xacro:macro>
-<!-- Links -->
-  <link name="base_link"/>
+  <!-- Links -->
+  <link name="base_link" />
   <link name="shell_link">
     <xacro:mesh_collision
       name="shell_collision"
-      mesh="${visual_mesh_dir}/Part__Feature001.010.dae"
+      mesh="${collision_mesh_dir}/Part__Feature001.010.stl"
       xyz="0.0000 0.0000 0.0000"
-      rpy="0.0000 0.0000 0.0000"/>
+      rpy="0.0000 0.0000 0.0000" />
     <xacro:link_inertial
       mass="0.5000"
@@ -68,5 +71,5 @@
       rpy="0.0000 0.0000 0.0000"
       ixx="0.0018" ixy="0.0000" ixz="-0.0007"
-      iyy="0.0027" iyz="0.0000" izz="0.0015"/>
+      iyy="0.0027" iyz="0.0000" izz="0.0015" />
     <xacro:mesh_visual
       name="shell"
@@ -74,12 +77,12 @@
       material="Part__Feature001.011"
       xyz="0.0000 0.0000 0.0000"
-      rpy="0.0000 0.0000 0.0000"/>
+      rpy="0.0000 0.0000 0.0000" />
   </link>
   <link name="neck_link">
     <xacro:mesh_collision
       name="neck_collision"
-      mesh="${visual_mesh_dir}/cgo3_vertical_arm_remeshed_v1.001.dae"
-      xyz="0.0000 -0.0000 0.0000"
-      rpy="0.0000 0.0000 0.0000"/>
+      mesh="${collision_mesh_dir}/cgo3_vertical_arm_remeshed_v1.001.stl"
+      xyz="0.0000 -0.0000 0.0000"
+      rpy="0.0000 0.0000 0.0000" />
     <xacro:link_inertial
       mass="0.0200"
@@ -87,5 +90,5 @@
       rpy="0.0000 0.0000 0.0000"
       ixx="0.0000043" ixy="0.0" ixz="0.0"
-      iyy="0.0000043" iyz="0.0" izz="0.0000003"/>
+      iyy="0.0000043" iyz="0.0" izz="0.0000003" />
     <xacro:mesh_visual
       name="neck"
@@ -93,12 +96,12 @@
       material="Material.003"
       xyz="0.0000 -0.0000 0.0000"
-      rpy="0.0000 0.0000 0.0000"/>
+      rpy="0.0000 0.0000 0.0000" />
   </link>
   <link name="neck_holder_link">
     <xacro:mesh_collision
       name="neck_holder_collision"
-      mesh="${visual_mesh_dir}/cgo3_horizontal_arm_remeshed_v1.001.stl"
-      xyz="0.0000 -0.0000 0.0000"
-      rpy="0.2104 -1.5708 -0.2104"/>
+      mesh="${collision_mesh_dir}/cgo3_horizontal_arm_remeshed_v1.001.stl"
+      xyz="0.0000 -0.0000 0.0000"
+      rpy="0.2104 -1.5708 -0.2104" />
     <xacro:link_inertial
       mass="0.0100"
@@ -106,5 +109,5 @@
       rpy="0.0000 0.0000 0.0000"
       ixx="0.0000031" ixy="0.0" ixz="0.0"
-      iyy="0.0000031" iyz="0.0" izz="0.0000001"/>
+      iyy="0.0000031" iyz="0.0" izz="0.0000001" />
     <xacro:mesh_visual
       name="neck_holder"
@@ -112,12 +115,12 @@
       material="green"
       xyz="0.0000 -0.0000 0.0000"
-      rpy="0.6040 -1.5708 -0.6040"/>
+      rpy="0.6040 -1.5708 -0.6040" />
   </link>
   <link name="camera_link">
     <xacro:mesh_collision
       name="camera_collision"
-      mesh="${visual_mesh_dir}/cgo3_camera_remeshed_v1.002.stl"
+      mesh="${collision_mesh_dir}/cgo3_camera_remeshed_v1.002.stl"
       xyz="0.0000 -0.0000 -0.0000"
-      rpy="-1.5708 0.0000 0.0000"/>
+      rpy="-1.5708 0.0000 0.0000" />
     <xacro:link_inertial
       mass="0.1000"
@@ -125,5 +128,5 @@
       rpy="0.0000 0.0000 0.0000"
       ixx="0.0000150" ixy="0.0" ixz="0.0"
-      iyy="0.0000150" iyz="0.0" izz="0.0000150"/>
+      iyy="0.0000150" iyz="0.0" izz="0.0000150" />
     <xacro:mesh_visual
       name="camera"
@@ -131,12 +134,12 @@
       material="Material.001"
       xyz="0.0000 -0.0000 -0.0000"
-      rpy="-1.5708 0.0000 0.0000"/>
+      rpy="-1.5708 0.0000 0.0000" />
   </link>
   <link name="feet_right_front_link">
     <xacro:mesh_collision
       name="feet_right_front_collision"
-      mesh="${visual_mesh_dir}/Part__Feature075.026.stl"
-      xyz="0.0000 -0.0000 0.0000"
-      rpy="1.5708 0.0000 0.0000"/>
+      mesh="${collision_mesh_dir}/Part__Feature075.026.stl"
+      xyz="0.0000 -0.0000 0.0000"
+      rpy="1.5708 0.0000 0.0000" />
     <xacro:link_inertial
       mass="0.2000"
@@ -144,5 +147,5 @@
       rpy="0.0000 0.0000 0.0000"
       ixx="0.0001" ixy="-0.0000" ixz="0.0000"
-      iyy="0.0002" iyz="0.0000" izz="0.0002"/>
+      iyy="0.0002" iyz="0.0000" izz="0.0002" />
     <xacro:mesh_visual
       name="feet_right_front"
@@ -150,12 +153,12 @@
       material="purple"
       xyz="0.0000 -0.0000 0.0000"
-      rpy="1.5708 0.0000 -0.0000"/>
+      rpy="1.5708 0.0000 -0.0000" />
   </link>
   <link name="wheel_right_front_link">
     <xacro:mesh_collision
       name="wheel_right_front_collision"
-      mesh="${visual_mesh_dir}/Part__Feature075.005.stl"
+      mesh="${collision_mesh_dir}/Part__Feature075.005.stl"
       xyz="-0.0001 -0.0002 0.0048"
-      rpy="1.5708 0.0000 0.0000"/>
+      rpy="1.5708 0.0000 0.0000" />
     <xacro:link_inertial
       mass="0.0400"
@@ -163,5 +166,5 @@
       rpy="0.0000 0.0000 0.0000"
       ixx="0.0000043" ixy="0.0" ixz="0.0"
-      iyy="0.0000043" iyz="0.0" izz="0.0000080"/>
+      iyy="0.0000043" iyz="0.0" izz="0.0000080" />
     <xacro:mesh_visual
       name="wheel_right_front"
@@ -169,12 +172,12 @@
       material="bones.001"
       xyz="-0.0001 -0.0002 0.0048"
-      rpy="1.5708 0.0000 0.0000"/>
+      rpy="1.5708 0.0000 0.0000" />
   </link>
   <link name="feet_right_rear_link">
     <xacro:mesh_collision
       name="feet_right_rear_collision"
-      mesh="${visual_mesh_dir}/Part__Feature075.027.stl"
+      mesh="${collision_mesh_dir}/Part__Feature075.027.stl"
       xyz="-0.0000 -0.0000 0.0000"
-      rpy="1.5708 0.0000 0.0000"/>
+      rpy="1.5708 0.0000 0.0000" />
     <xacro:link_inertial
       mass="0.2000"
@@ -182,5 +185,5 @@
       rpy="0.0000 0.0000 0.0000"
       ixx="0.0001" ixy="0.0000" ixz="-0.0000"
-      iyy="0.0002" iyz="0.0000" izz="0.0002"/>
+      iyy="0.0002" iyz="0.0000" izz="0.0002" />
     <xacro:mesh_visual
       name="feet_right_rear"
@@ -188,12 +191,12 @@
       material="purple"
       xyz="-0.0000 -0.0000 0.0000"
-      rpy="1.5708 0.0000 0.0000"/>
+      rpy="1.5708 0.0000 0.0000" />
   </link>
   <link name="wheel_right_rear_link">
     <xacro:mesh_collision
       name="wheel_right_rear_collision"
-      mesh="${visual_mesh_dir}/Part__Feature075.001.stl"
+      mesh="${collision_mesh_dir}/Part__Feature075.001.stl"
       xyz="0.0001 -0.0000 -0.0000"
-      rpy="1.5708 0.0000 0.0000"/>
+      rpy="1.5708 0.0000 0.0000" />
     <xacro:link_inertial
       mass="0.0400"
@@ -201,5 +204,5 @@
       rpy="0.0000 0.0000 0.0000"
       ixx="0.0000043" ixy="0.0" ixz="0.0"
-      iyy="0.0000043" iyz="0.0" izz="0.0000080"/>
+      iyy="0.0000043" iyz="0.0" izz="0.0000080" />
     <xacro:mesh_visual
       name="wheel_right_rear"
@@ -207,12 +210,12 @@
       material="wheels_material"
       xyz="0.0001 -0.0000 -0.0000"
-      rpy="1.5708 0.0000 0.0000"/>
+      rpy="1.5708 0.0000 0.0000" />
   </link>
   <link name="feet_left_rear_link">
     <xacro:mesh_collision
       name="feet_left_rear_collision"
-      mesh="${visual_mesh_dir}/Part__Feature075.028.stl"
+      mesh="${collision_mesh_dir}/Part__Feature075.028.stl"
       xyz="-0.0000 0.0000 0.0000"
-      rpy="-1.5708 0.0000 -0.0000"/>
+      rpy="-1.5708 0.0000 -0.0000" />
     <xacro:link_inertial
       mass="0.2000"
@@ -220,5 +223,5 @@
       rpy="0.0000 0.0000 0.0000"
       ixx="0.0001" ixy="-0.0000" ixz="-0.0000"
-      iyy="0.0002" iyz="-0.0000" izz="0.0002"/>
+      iyy="0.0002" iyz="-0.0000" izz="0.0002" />
     <xacro:mesh_visual
       name="feet_left_rear"
@@ -226,12 +229,12 @@
       material="purple"
       xyz="-0.0000 0.0000 0.0000"
-      rpy="-1.5708 0.0000 0.0000"/>
+      rpy="-1.5708 0.0000 0.0000" />
   </link>
   <link name="wheel_left_rear_link">
     <xacro:mesh_collision
       name="wheel_left_rear_collision"
-      mesh="${visual_mesh_dir}/Part__Feature075.020.stl"
+      mesh="${collision_mesh_dir}/Part__Feature075.020.stl"
       xyz="0.0000 -0.0003 0.0053"
-      rpy="-1.5708 0.0000 0.0000"/>
+      rpy="-1.5708 0.0000 0.0000" />
     <xacro:link_inertial
       mass="0.0400"
@@ -239,5 +242,5 @@
       rpy="0 0 0"
       ixx="0.0000043" ixy="0.0" ixz="0.0"
-      iyy="0.0000043" iyz="0.0" izz="0.0000080"/>
+      iyy="0.0000043" iyz="0.0" izz="0.0000080" />
     <xacro:mesh_visual
       name="wheel_left_rear"
@@ -245,12 +248,12 @@
       material="Part__Feature074.001"
       xyz="0.0000 -0.0003 0.0053"
-      rpy="-1.5708 0.0000 0.0000"/>
+      rpy="-1.5708 0.0000 0.0000" />
   </link>
   <link name="feet_left_front_link">
     <xacro:mesh_collision
       name="feet_left_front_collision"
-      mesh="${visual_mesh_dir}/Part__Feature075.008.stl"
+      mesh="${collision_mesh_dir}/Part__Feature075.008.stl"
       xyz="0.0000 0.0000 0.0000"
-      rpy="-1.5708 0.0000 0.0000"/>
+      rpy="-1.5708 0.0000 0.0000" />
     <xacro:link_inertial
       mass="0.2000"
@@ -258,5 +261,5 @@
       rpy="0.0000 0.0000 0.0000"
       ixx="0.0001" ixy="0.0000" ixz="0.0000"
-      iyy="0.0002" iyz="-0.0000" izz="0.0002"/>
+      iyy="0.0002" iyz="-0.0000" izz="0.0002" />
     <xacro:mesh_visual
       name="node131.004"
@@ -264,5 +267,5 @@
       material="purple"
       xyz="0.0000 0.0000 0.0000"
-      rpy="-1.5708 0.0000 0.0000"/>
+      rpy="-1.5708 0.0000 0.0000" />
     <xacro:mesh_visual
       name="feet_left_front"
@@ -270,12 +273,12 @@
       material="purple"
       xyz="0.0000 0.0000 0.0000"
-      rpy="-1.5708 0.0000 0.0000"/>
+      rpy="-1.5708 0.0000 0.0000" />
   </link>
   <link name="wheel_left_front_link">
     <xacro:mesh_collision
       name="wheel_left_front_collision"
-      mesh="${visual_mesh_dir}/Part__Feature075.019.stl"
+      mesh="${collision_mesh_dir}/Part__Feature075.019.stl"
       xyz="-0.0001 0.0001 0.0053"
-      rpy="-1.5708 0.0000 0.0000"/>
+      rpy="-1.5708 0.0000 0.0000" />
     <xacro:link_inertial
       mass="0.0400"
@@ -283,5 +286,5 @@
       rpy="0.0000 0.0000 0.0000"
       ixx="0.0000043" ixy="0.0" ixz="0.0"
-      iyy="0.0000043" iyz="0.0" izz="0.0000080"/>
+      iyy="0.0000043" iyz="0.0" izz="0.0000080" />
     <xacro:mesh_visual
       name="wheel_left_front"
@@ -289,7 +292,7 @@
       material="Part__Feature074.001"
       xyz="-0.0001 0.0001 0.0053"
-      rpy="-1.5708 0.0000 0.0000"/>
-  </link>
-<!-- Joints -->
+      rpy="-1.5708 0.0000 0.0000" />
+  </link>
+  <!-- Joints -->
   <xacro:fixed_joint
     name="base_to_body"
@@ -297,5 +300,5 @@
     child="shell_link"
     xyz="0 0 0"
-    rpy="0 0 0"/>
+    rpy="0 0 0" />
   <xacro:revolute_joint
     name="neck_link_joint"
@@ -306,5 +309,5 @@
     axis="0.0000 0.0000 1.0000"
     lower="-3.1400" upper="3.1400"
-    effort="0.0000" velocity="0.0000"/>
+    effort="0.0000" velocity="0.0000" />
   <xacro:revolute_joint
     name="neck_holder_link_joint"
@@ -315,5 +318,5 @@
     axis="0.0000 0.0000 1.0000"
     lower="-3.1400" upper="3.1400"
-    effort="0.0000" velocity="0.0000"/>
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
File: roma_gazebo/urdf/roma_gz.urdf.xacro (robot description, xacro)
@@ -1,5 +1,4 @@
 <?xml version="1.0"?>
 <robot name="roma" xmlns:xacro="http://www.ros.org/wiki/xacro">
-    <xacro:include filename="$(find roma_description)/urdf/roma.urdf.xacro"/>
-    <xacro:include filename="$(find roma_gazebo)/urdf/robot_material_support.xacro"/>
+    <xacro:include filename="$(find-pkg-share roma_description)/urdf/roma.urdf.xacro"/>
 </robot>

Commit message: feat: gz bridge plus teleop twist

File: roma_description/urdf/roma.urdf (robot description, URDF)
Before this commit: robot roma, 13 links, 12 joints
Links:
- link shell_link: geometry collision box size=0.21 0.12 0.14; visual mesh filename=package://roma_description/meshes/visual/Part__Feature001.0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 scale=1 1 1

File: roma_description/urdf/roma.urdf.xacro (robot description, xacro)
@@ -58,12 +58,20 @@
     </joint>
   </xacro:macro>
+  <xacro:macro name="box_collision" params="name size xyz rpy">
+    <collision name="${name}">
+      <origin xyz="${xyz}" rpy="${rpy}" />
+      <geometry>
+        <box size="${size}" />
+      </geometry>
+    </collision>
+  </xacro:macro>
   <!-- Links -->
   <link name="base_link" />
   <link name="shell_link">
-    <xacro:mesh_collision
+    <xacro:box_collision
       name="shell_collision"
-      mesh="${collision_mesh_dir}/Part__Feature001.010.stl"
       xyz="0.0000 0.0000 0.0000"
-      rpy="0.0000 0.0000 0.0000" />
+      rpy="0.0000 0.0000 0.0300"
+      size="0.21 0.12 0.04" />
     <xacro:link_inertial
       mass="0.5000"
@@ -328,13 +336,13 @@
     lower="-3.1400" upper="3.1400"
     effort="0.0000" velocity="0.0000" />
-  <xacro:revolute_joint
+  <xacro:fixed_joint
     name="feet_right_rear_link_joint"
     parent="shell_link"
     child="feet_right_rear_link"
     xyz="0.0476 0.0521 -0.0565"
-    rpy="-1.5708 0.0000 0.0000"
-    axis="0.0000 0.0000 -1.0000"
-    lower="-3.1400" upper="3.1400"
-    effort="0.0000" velocity="0.0000" />
+    rpy="-1.5708 0.0000 0.0000" />
+  <!-- axis="0.0000 0.0000 -1.0000"
+    lower="-3.1400" upper="3.1400"
+    effort="0.0000" velocity="0.0000"  -->
   <xacro:continuous_joint
     name="wheel_right_rear_link_joint"
@@ -345,13 +353,13 @@
     axis="0.0000 0.0000 -1.0000"
     effort="10.0000" velocity="20.0000" />
-  <xacro:revolute_joint
+  <xacro:fixed_joint
     name="feet_left_rear_link_joint"
     parent="shell_link"
     child="feet_left_rear_link"
     xyz="0.0476 -0.0522 -0.0565"
-    rpy="1.5708 0.0000 -0.0000"
-    axis="0.0000 0.0000 1.0000"
-    lower="-3.1400" upper="3.1400"
-    effort="0.0000" velocity="0.0000" />
+    rpy="1.5708 0.0000 -0.0000" />
+  <!-- axis="0.0000 0.0000 1.0000"
+    lower="-3.1400" upper="3.1400"
+    effort="0.0000" velocity="0.0000"  -->
   <xacro:continuous_joint
     name="wheel_left_rear_link_joint"
@@ -362,13 +370,13 @@
     axis="0.0000 0.0000 1.0000"
     effort="10.0000" velocity="20.0000" />
-  <xacro:revolute_joint
+  <xacro:fixed_joint
     name="feet_left_front_link_joint"
     parent="shell_link"
     child="feet_left_front_link"
     xyz="-0.0479 -0.0522 -0.0565"
-    rpy="1.5708 0.0000 -0.0000"
-    axis="0.0000 0.0000 1.0000"
-    lower="-3.1400" upper="3.1400"
-    effort="0.0000" velocity="0.0000" />
+    rpy="1.5708 0.0000 -0.0000" />
+  <!-- axis="0.0000 0.0000 1.0000"
+    lower="-3.1400" upper="3.1400"
+    effort="0.0000" velocity="0.0000"  -->
   <xacro:continuous_joint
     name="wheel_left_front_link_joint"
@@ -379,13 +387,13 @@
     axis="0.0000 0.0000 1.0000"
     effort="10.0000" velocity="20.0000" />
-  <xacro:revolute_joint
+  <xacro:fixed_joint
     name="feet_right_front_link_joint"
     parent="shell_link"
     child="feet_right_front_link"
     xyz="-0.0479 0.0522 -0.0565"
-    rpy="-1.5708 0.0000 -0.0000"
-    axis="0.0000 0.0000 -1.0000"
-    lower="-3.1400" upper="3.1400"
-    effort="0.0000" velocity="0.0000" />
+    rpy="-1.5708 0.0000 -0.0000" />
+  <!-- axis="0.0000 0.0000 -1.0000"
+    lower="-3.1400" upper="3.1400"
+    effort="0.0000" velocity="0.0000"  -->
   <xacro:continuous_joint
     name="wheel_right_front_link_joint"
@@ -396,31 +404,39 @@
     axis="0.0000 0.0000 -1.0000"
     effort="10.0000" velocity="20.0000" />
-  <!-- Materiales -->
-  <material name="gray">
-    <color rgba="0.5 0.5 0.5 1.0" />
-  </material>
-  <material name="Material.001">
-    <color rgba="0.1804 0.0000 0.0000 1.0000" />
-  </material>
-  <material name="Material.003">
-    <color rgba="0.0000 0.0000 0.1098 1.0000" />
-  </material>
-  <material name="Part__Feature001.011">
-    <color rgba="0.0000 0.5961 0.0078 1.0000" />
-  </material>
-  <material name="Part__Feature074.001">
-    <color rgba="0.2941 0.2745 0.0000 1.0000" />
-  </material>
-  <material name="bones.001">
-    <color rgba="0.0000 0.0000 0.0000 1.0000" />
-  </material>
-  <material name="green">
-    <color rgba="0.0902 0.0000 0.0863 1.0000" />
-  </material>
-  <material name="purple">
-    <color rgba="0.0314 0.0039 0.0275 1.0000" />
-  </material>
-  <material name="wheels_material">
-    <color rgba="0.0000 0.0000 0.0000 1.0000" />
-  </material>
+  <!-- ===== Gazebo Plugins ===== -->
+  <!-- Plugin 1: Differential Drive-->
+  <gazebo>
+    <plugin filename="gz-sim-diff-drive-system"
+      name="gz::sim::systems::DiffDrive">
+      <!-- Ruedas izquierdas -->
+      <left_joint>wheel_left_front_link_joint</left_joint>
+      <left_joint>wheel_left_rear_link_joint</left_joint>
+      <!-- Ruedas derechas -->
+      <right_joint>wheel_right_front_link_joint</right_joint>
+      <right_joint>wheel_right_rear_link_joint</right_joint>
+      <!-- Geometría del robot -->
+      <wheel_separation>0.1048</wheel_separation>
+      <wheel_radius>0.020</wheel_radius>
+      <!-- Tópicos -->
+      <topic>cmd_vel</topic>
+      <odom_topic>odom</odom_topic>
+      <frame_id>odom</frame_id>
+      <child_frame_id>base_link</child_frame_id>
+      <odom_publish_frequency>50</odom_publish_frequency>
+      <tf_topic>/tf</tf_topic>
+    </plugin>
+  </gazebo>
+  <!-- Plugin 2: Publicar estado de joints -->
+  <gazebo>
+    <plugin filename="gz-sim-joint-state-publisher-system"
+      name="gz::sim::systems::JointStatePublisher">
+      <topic>joint_states</topic>
+      <left_joint>wheel_left_front_link_joint</left_joint>
+      <left_joint>wheel_left_rear_link_joint</left_joint>
+      <!-- Ruedas derechas -->
+      <right_joint>wheel_right_front_link_joint</right_joint>
+      <right_joint>wheel_right_rear_link_joint</right_joint>
+    </plugin>
+  </gazebo>
+  <xacro:include filename="$(find roma_gazebo)/urdf/robot_material_support.xacro" />
 </robot>

File: roma_gazebo/urdf/roma_gz.urdf.xacro (robot description, xacro)
@@ -1,4 +1,4 @@
 <?xml version="1.0"?>
 <robot name="roma" xmlns:xacro="http://www.ros.org/wiki/xacro">
-    <xacro:include filename="$(find-pkg-share roma_description)/urdf/roma.urdf.xacro"/>
+    <xacro:include filename="$(find roma_description)/urdf/roma.urdf.xacro" />
 </robot>
