Commit message: feat: implement SLAM as first step toward nav2 (casi que no xd)

File: roma_gazebo/urdf/robot_material_support.xacro (robot description, xacro)
@@ -1,30 +1,30 @@
 <?xml version="1.0"?>
-<robot xmlns:xacro="http://www.ros.org/wiki/xacro" >
-<material name="gray">
-    <color rgba="0.5 0.5 0.5 1.0"/>
+<robot xmlns:xacro="http://www.ros.org/wiki/xacro">
+  <material name="gray">
+    <color rgba="0.5 0.5 0.5 1.0" />
   </material>
   <material name="Material.001">
-    <color rgba="0.1804 0.0000 0.0000 1.0000"/>
+    <color rgba="0.1804 0.0000 0.0000 1.0000" />
   </material>
   <material name="Material.003">
-    <color rgba="0.0000 0.0000 0.1098 1.0000"/>
+    <color rgba="0.0000 0.0000 0.1098 1.0000" />
   </material>
   <material name="Part__Feature001.011">
-    <color rgba="0.0000 0.5961 0.0078 1.0000"/>
+    <color rgba="0.0000 0.5961 0.0078 1.0000" />
   </material>
   <material name="Part__Feature074.001">
-    <color rgba="0.2941 0.2745 0.0000 1.0000"/>
+    <color rgba="0.2941 0.2745 0.0000 1.0000" />
   </material>
   <material name="bones.001">
-    <color rgba="0.0000 0.0000 0.0000 1.0000"/>
+    <color rgba="0.0000 0.0000 0.0000 1.0000" />
   </material>
   <material name="green">
-    <color rgba="0.0902 0.0000 0.0863 1.0000"/>
+    <color rgba="0.0902 0.0000 0.0863 1.0000" />
   </material>
   <material name="purple">
-    <color rgba="0.0314 0.0039 0.0275 1.0000"/>
+    <color rgba="0.0314 0.0039 0.0275 1.0000" />
   </material>
   <material name="wheels_material">
-    <color rgba="0.0000 0.0000 0.0000 1.0000"/>
+    <color rgba="0.0000 0.0000 0.0000 1.0000" />
   </material>
 </robot>

File: roma_gazebo/urdf/roma_gz.urdf.xacro (robot description, xacro)
@@ -6,6 +6,7 @@
             <always_on>true</always_on>
             <visualize>true</visualize>
-            <update_rate>5</update_rate>
-            <topic>scan</topic>
+            <update_rate>10</update_rate>
+            <topic>/scan</topic>
+            <frame_id>camera_link</frame_id>
             <gz_frame_id>camera_link</gz_frame_id>
             <ray>
@@ -13,13 +14,19 @@
                     <horizontal>
                         <samples>360</samples>
-                        <resolution>1.000000</resolution>
-                        <min_angle>0.000000</min_angle>
-                        <max_angle>6.280000</max_angle>
+                        <resolution>1</resolution>
+                        <min_angle>-3.14159</min_angle>
+                        <max_angle>3.14159</max_angle>
                     </horizontal>
+                    <vertical>
+                        <samples>1</samples>
+                        <resolution>1</resolution>
+                        <min_angle>0</min_angle>
+                        <max_angle>0</max_angle>
+                    </vertical>
                 </scan>
                 <range>
-                    <min>0.120000</min>
+                    <min>0.12</min>
                     <max>3.5</max>
-                    <resolution>0.015000</resolution>
+                    <resolution>0.015</resolution>
                 </range>
                 <noise>
@@ -31,8 +38,3 @@
         </sensor>
     </gazebo>
-    <gazebo>
-        <plugin filename="gz-sim-sensors-system" name="gz::sim::systems::Sensors">
-            <render_engine>ogre2</render_engine>
-        </plugin>
-    </gazebo>
 </robot>
